File: MainBoard/mainboard.kicad_sch (KiCad schematic)
At the start: 4 parts

Commit message: Add logo and update project variables
Changed lines of the file:
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@@
 		(company "${Company}")
+	)
+	(polyline
+		(pts
+			(xy 272.8407 174.5096) (xy 272.8147 177.2941) (xy 272.0248 178.1148) (xy 270.3008 178.1307) (xy 270.3529 177.402)
+			(xy 270.9514 176.9076) (xy 270.3345 176.3308) (xy 270.3221 174.4966) (xy 272.8407 174.5096)
+		)
+		(stroke
+			(width -0.0001)
+			(type solid)
+		)
+		(fill
+			(type outline)
+		)
+	)
+	(polyline
+		(pts
+			(xy 278.1253 171.5784) (xy 278.0891 173.0109) (xy 278.0716 173.494) (xy 278.0563 173.6946) (xy 278.0512 173.701)
+			(xy 278.043 173.7065) (xy 278.0319 173.7111) (xy 278.0181 173.7149) (xy 277.9832 173.7202) (xy 277.9402 173.7228)
+			(xy 277.8906 173.7229) (xy 277.8364 173.7211) (xy 277.7205 173.713) (xy 277.6064 173.7014) (xy 277.5077 173.6894)
+			(xy 277.4123 173.6762) (xy 277.5411 169.5359) (xy 278.1667 169.5175) (xy 278.1253 171.5784)
+		)
+		(stroke
+			(width -0.0001)
+			(type solid)
+		)
+		(fill
+			(type outline)
+		)
+	)
+	(polyline
+		(pts
+			(xy 274.1624 174.5556) (xy 275.0472 175.3075) (xy 275.0472 174.5946) (xy 275.8539 174.5686) (xy 275.945 178.0491)
+			(xy 275.1123 178.0751) (xy 274.2106 177.4086) (xy 274.2014 178.0751) (xy 273.4467 178.1271) (xy 273.4337 174.5296)
+			(xy 274.1624 174.5556)
+		)
+		(stroke
+			(width -0.0001)
+			(type solid)
+		)
+		(fill
+			(type outline)
+		)
+	)
+	(polyline
+		(pts
+			(xy 281.2981 170.4927) (xy 280.7277 171.008) (xy 281.3073 171.6244) (xy 281.2981 173.0321) (xy 280.6909 173.6578)
+			(xy 278.8139 173.6762) (xy 278.8323 172.9585) (xy 279.366 172.4065) (xy 278.8047 171.9005) (xy 278.8508 170.1431)
+			(xy 279.4028 169.5727) (xy 280.3597 169.5575) (xy 280.8502 169.548) (xy 281.3165 169.5359) (xy 281.2981 170.4927)
+		)
+		(stroke
+			(width -0.0001)
+			(type solid)
+		)
+		(fill
+			(type outline)
+		)
+	)
+	(polyline
+		(pts
+			(xy 281.1915 178.1115) (xy 280.671 178.1115) (xy 280.0464 177.2007) (xy 279.604 178.0074) (xy 278.9014 178.0855)
+			(xy 278.9858 174.6969) (xy 279.5323 174.6969) (xy 280.1308 175.5817) (xy 280.6252 174.6188) (xy 281.2758 174.5667)
+			(xy 281.1915 178.1115)
+		)
+		(stroke
+			(width -0.0001)
+			(type solid)
+		)
+		(fill
+			(type outline)
+		)
+	)
+	(polyline
+		(pts
+			(xy 269.6902 170.2688) (xy 269.5982 172.845) (xy 268.4389 173.6178) (xy 266.4883 173.5994) (xy 266.5619 169.2751)
+			(xy 268.8805 169.2383) (xy 269.6902 170.2688)
+		)
+		(stroke
+			(width -0.0001)
+			(type solid)
+		)
+		(fill
+			(type outline)
+		)
+	)
+	(polyline
+		(pts
+			(xy 276.1286 169.5035) (xy 276.7911 170.074) (xy 276.7543 171.4541) (xy 275.7054 172.3558) (xy 276.6439 173.6991)
+			(xy 274.0677 173.6991) (xy 274.0884 171.5622) (xy 274.1065 170.0737) (xy 274.1229 169.3563) (xy 276.1286 169.5035)
+		)
+		(stroke
+			(width -0.0001)
+			(type solid)
+		)
+		(fill
+			(type outline)
+		)
+	)
+	(polyline
+		(pts
+			(xy 269.6944 175.2113) (xy 269.0438 175.7057) (xy 269.6944 176.1742) (xy 269.6684 177.6533) (xy 269.0699 178.2779)
+			(xy 266.5976 178.3039) (xy 266.6236 177.5492) (xy 267.2117 177.0193) (xy 266.6328 176.5416) (xy 266.6389 175.1737)
+			(xy 267.2742 174.5045) (xy 269.6944 174.5044) (xy 269.6944 175.2113)
+		)
+		(stroke
+			(width -0.0001)
+			(type solid)
+		)
+		(fill
+			(type outline)
+		)
+	)
+	(polyline
+		(pts
+			(xy 278.572 174.6695) (xy 278.5781 175.343) (xy 277.7913 175.8842) (xy 277.7133 178.0042) (xy 276.9523 178.0455)
+			(xy 276.9951 175.8919) (xy 276.3531 175.395) (xy 276.3531 174.6664) (xy 278.572 174.6695)
+		)
+		(stroke
+			(width -0.0001)
+			(type solid)
+		)
+		(fill
+			(type outline)
+		)
+	)
+	(polyline
+		(pts
+			(xy 279.4028 169.5727) (xy 279.4028 169.5727)
+		)
+		(stroke
+			(width -0.0001)
+			(type solid)
+		)
+		(fill
+			(type outline)
+		)
+	)
+	(polyline
+		(pts
+			(xy 272.8608 169.4299) (xy 273.3392 170.166) (xy 273.284 173.1654) (xy 272.732 173.6991) (xy 270.8366 173.6991)
+			(xy 270.2294 172.9262) (xy 270.3398 170.0924) (xy 271.1127 169.2275) (xy 272.8608 169.4299)
+		)
+		(stroke
+			(width -0.0001)
+			(type solid)
+		)
+		(fill
+			(type outline)
+		)
 	)
 	(wire
@@
 		)
 		(instances
-			(project "mainboard"
+			(project "MainBoard"
 				(path "/9e709b97-b403-4027-b7d8-a3ed3b3557e2"
 					(page "4")
@@
 		)
 		(instances
-			(project "mainboard"
+			(project "MainBoard"
 				(path "/9e709b97-b403-4027-b7d8-a3ed3b3557e2"
 					(page "4")
@@
 		)
 		(instances
-			(project "mainboard"
+			(project "MainBoard"
 				(path "/9e709b97-b403-4027-b7d8-a3ed3b3557e2"
 					(page "2")
