File: MatrixBoard/MatrixBoard.kicad_pcb (KiCad board)
At the start: 2 copper layers, 40 x 32 mm, 130 parts, among them J1 MATRIX_IN, J2 MATRIX_OUT

Commit message: Udpate project variables and add texts
Other:
- board text added: "${PROJECTNAME}"
Changed lines of the file:
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@@
+		)
+	)
+	(gr_text "${PROJECTNAME}"
+		(at 164 100.5 0)
+		(layer "B.SilkS")
+		(effects
+			(font
+				(size 1 1)
+				(thickness 0.1)
+			)
+			(justify bottom mirror)
 		)
 	)

Commit message: Add logo and update project variables
Other:
- board text added: "${Revision}"
- board text removed: "${REVISION}"
Changed lines of the file:
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@@
 	(paper "A4")
 	(title_block
-		(title "VirtualBlob")
-		(date "2025-11-10")
-		(rev "${revision}")
-		(company "Miłosz Derżko")
+		(title "${ProjectTitle}")
+		(date "2025-11-23")
+		(rev "${Revision}")
+		(company "${Company}")
 	)
 	(layers
@@
 		)
 	)
+	(gr_poly
+		(pts
+			(xy 165.292846 107.004283) (xy 165.053626 107.372313) (xy 165.081228 108.872034) (xy 165.357251 109.138855)
+			(xy 166.304927 109.138855) (xy 166.608552 108.752424) (xy 166.553347 107.335509) (xy 166.166916 106.903075)
+		)
+		(stroke
+			(width 0)
+			(type solid)
+		)
+		(fill yes)
+		(layer "B.SilkS")
+	)
+	(gr_poly
+		(pts
+			(xy 161.294986 107.535693) (xy 161.58021 107.793314) (xy 161.290387 108.101539) (xy 161.294988 108.805396)
+			(xy 161.598613 109.118221) (xy 162.537088 109.127422) (xy 162.527887 108.768593) (xy 162.261065 108.492571)
+			(xy 162.541688 108.23955) (xy 162.518686 107.36088) (xy 162.242664 107.075656) (xy 162.242663 107.075656)
+			(xy 161.76419 107.068053) (xy 161.518935 107.063345) (xy 161.285786 107.057254)
+		)
+		(stroke
+			(width 0)
+			(type solid)
+		)
+		(fill yes)
+		(layer "B.SilkS")
+	)
+	(gr_poly
+		(pts
+			(xy 162.83539 108.050935) (xy 162.853504 108.767156) (xy 162.862237 109.008711) (xy 162.869893 109.109021)
+			(xy 162.872435 109.112232) (xy 162.876541 109.114982) (xy 162.882103 109.117294) (xy 162.889013 109.119192)
+			(xy 162.906444 109.121838) (xy 162.927972 109.123109) (xy 162.952735 109.123194) (xy 162.97987 109.122282)
+			(xy 163.037806 109.118221) (xy 163.094879 109.112435) (xy 163.14419 109.106433) (xy 163.191919 109.09982)
+			(xy 163.127514 107.029652) (xy 162.814688 107.020452)
+		)
+		(stroke
+			(width 0)
+			(type solid)
+		)
+		(fill yes)
+		(layer "B.SilkS")
+	)
+	(gr_poly
+		(pts
+			(xy 159.688526 107.431274) (xy 159.927993 107.683753) (xy 159.680114 107.991706) (xy 159.668681 108.757418)
+			(xy 159.993976 109.095726) (xy 160.956851 109.108738) (xy 160.94305 108.65161) (xy 160.659812 108.385195)
+			(xy 160.949229 108.14336) (xy 160.948439 107.363057) (xy 160.714226 107.050774) (xy 159.692337 107.03014)
+		)
+		(stroke
+			(width 0)
+			(type solid)
+		)
+		(fill yes)
+		(layer "B.SilkS")
+	)
+	(gr_poly
+		(pts
+			(xy 163.760133 107.031885) (xy 163.428906 107.317108) (xy 163.447307 108.007164) (xy 163.97175 108.458)
+			(xy 163.502512 109.129654) (xy 164.790616 109.129654) (xy 164.780265 108.061218) (xy 164.771208 107.316964)
+			(xy 164.763014 106.958279)
+		)
+		(stroke
+			(width 0)
+			(type solid)
+		)
+		(fill yes)
+		(layer "B.SilkS")
+	)
+	(gr_poly
+		(pts
+			(xy 166.78614 107.405304) (xy 166.832144 108.693409) (xy 167.411791 109.07984) (xy 168.387069 109.070639)
+			(xy 168.350267 106.908464) (xy 167.190973 106.890063)
+		)
+		(stroke
+			(width 0)
+			(type solid)
+		)
+		(fill yes)
+		(layer "B.SilkS")
+	)
 	(gr_arc
 		(start 146 120)
@@
 		)
 	)
-	(gr_text "${REVISION}"
+	(gr_text "${Revision}"
 		(at 164.084 104.648 0)
 		(layer "B.SilkS")
@@
 		)
 	)
+	(group ""
+		(members "21e0fc2c-15f1-4aca-a19f-c9d3db477a32" "860cd7a4-45c1-4d80-bcf6-9bf6ed25ae94"
+			"86e7dab6-1356-4920-827e-1d13c4df50ca" "b122d52e-ce2c-41b8-b28c-2c2d9298fad8"
+			"b2e2a8e5-7c7b-4c5d-92b5-b146d7a9787d" "cabbee00-158b-4033-a042-084e2a4e9724"
+		)
+	)
