File: MatrixBoard/Row.kicad_sch (KiCad schematic)
At the start: 16 parts

Commit message: add new spring touch
Other:
- company: Miłosz Derżko -> ${Company}
- title: VirtualBlob -> ${ProjectTitle}
Changed lines of the file:
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@@
 	(paper "A4")
 	(title_block
-		(title "VirtualBlob")
+		(title "${ProjectTitle}")
 		(date "2025-11-10")
-		(rev "${revision}")
-		(company "Miłosz Derżko")
+		(rev "${Revision}")
+		(company "${Company}")
 	)
 	(junction
